File: circuits/lightclock.0/lightclock.0.brd (EAGLE design)
At the start: 38.1 x 38.1 mm, 44 parts, among them J1 USB-MINI-651005136421, J10 TESTPAD, J11 TESTPAD, J12 TESTPAD, J13 TESTPAD, J14 TESTPAD, J15 TESTPAD, J16 TESTPAD, J17 TESTPAD, J2 TESTPAD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

Commit message: almost done with layout, just needs a review
Parts:
- added J18, J19, J20, J21: TESTPAD, Kemper-Connectors:HEADER-1X1
- moved J3 10.2 mm to (25.4, 35.6)
- moved J4 10.2 mm to (22.9, 35.6)
- moved J5 10.2 mm to (20.3, 35.6)
- moved J6 10.2 mm to (17.8, 35.6)
- moved J8 10.2 mm to (12.7, 35.6)
- moved J7 10.2 mm to (15.2, 35.6)
- moved J2 8.03 mm to (27.9, 35.6)
- moved J9 5.24 mm to (35.6, 3.81), turned to 180 degrees
- moved S1 1.27 mm to (15.0, 31.2)
Connections:
- net +3V3: now also J18.1, J20.1
- net GND: now also J19.1, J21.1
Routing:
- net N$13: track 3.54 -> 12.5 mm
- net N$11: track 3.76 -> 10.8 mm
- net N$14: track 3.82 -> 10.7 mm
- net N$15: track 4.69 -> 8.93 mm
- net N$17: track 8.21 -> 5.70 mm
- net N$18: track 6.59 -> 4.09 mm
- net PDI_DATA: track 25.3 -> 23.7 mm
- net N$16: track 6.45 -> 7.47 mm
- net GND: track 30.4 -> 31.3 mm, vias 11 -> 10
- net SWITCH: track 19.8 -> 20.5 mm
- net PDI_CLK: track 18.1 -> 18.7 mm
Other:
- board text added: "C3"
- board text added: "C7"
- board text added: "GND"

Commit message: final lightclock.0
Routing:
- net BT_RESET: track 53.0 -> 53.8 mm
Other:
- board size 38.1 x 38.1 mm -> 38.4 x 38.4 mm
- board text added: "59354"
